Commit message: -Moving the project into rviz only, without gazebo -Adjusting a lot of the launch and description

File: project_description/urdf/irb120_gripper/irb120_gripper.xacro (robot description, xacro)
@@ -1,6 +1,11 @@
 <?xml version="1.0"?>
 <robot xmlns:xacro="http://ros.org/wiki/xacro" name="irb120_assembly">
+  <!-- 1. Include Robot Arm Macro -->
   <xacro:include filename="$(find project_description)/urdf/irb120_3_58/irb120_3_58_macro.xacro"/>
+  <!-- 2. Include Gripper Macro -->
   <xacro:include filename="$(find project_description)/urdf/2fg7/onrobot_2fg7.xacro"/>
+  <!-- 3. Include Taskboard Environment URDF -->
+  <xacro:include filename="$(find project_description)/urdf/taskboard/taskboard_environment.urdf"/>
+  <!-- 4. Base World Link & Fixed Joint to Robot Base -->
   <link name="world" />
   <joint name="world_to_robot" type="fixed">
@@ -9,13 +14,9 @@
     <origin xyz="0 0.32 0" rpy="0 0 0" />
   </joint>
+  <!-- 5. Instantiate ABB IRB 120 -->
   <xacro:abb_irb120_3_58 prefix=""/>
-  <xacro:onrobot_2fg7 prefix="gripper_" parent="tool0">
+  <!-- 6. Instantiate OnRobot 2FG7 attached to tool0 -->
+  <xacro:onrobot_2fg7 prefix="" parent="tool0">
     <origin xyz="0 0 0" rpy="0 0 0" />
   </xacro:onrobot_2fg7>
-  <xacro:onrobot_2fg7_fingertip prefix="right_" parent="gripper_right_attachment" side="right">
-    <origin xyz="0 0 0" rpy="0 0 3.14159265359"/>
-  </xacro:onrobot_2fg7_fingertip>
-  <xacro:onrobot_2fg7_fingertip prefix="left_" parent="gripper_left_attachment" side="left">
-      <origin xyz="0 0 0" rpy="0 0 0"/>
-  </xacro:onrobot_2fg7_fingertip>
 </robot>
