Commit message: -Continuing the assembly

File: project_description/urdf/irb1200_5_90/irb1200_5_90.urdf (robot description, URDF)
Before this commit: robot abb_irb1200_5_90, 11 links, 10 joints
Links:
- removed link base
- removed link flange
- removed link world
- link tool0: mass None -> 0.0001
Joints:
- removed joint base_link-base
- removed joint joint_6-flange
- removed joint link_6-tool0
- removed joint world_fixed
- added joint tool0_joint: type fixed, parent link_6, child tool0, origin xyz=0 0 0 rpy=0 1.5707963267948966 0

File: project_description/urdf/irb120_3_58/irb120_3_58_robot.urdf (robot description, URDF)
Before this commit: robot irb120_assembly, 11 links, 10 joints
Joints:
- joint gripper_gripper_joint: limit lower=0.0 upper=0.038 effort=100 velocity=0.1 -> lower=0.0 upper=0.009 effort=100 velocity=0.1
- joint gripper_right_joint: axis (none) -> 1 0 0; limit (none) -> lower=0.0 upper=0.009 effort=100 velocity=0.1; mimic (none) -> joint=gripper_gripper_joint multiplier=1.0; type fixed -> prismatic

File: project_description/urdf/irb120_3_58/irb120_3_58_taskboard.urdf (robot description, URDF)
Before this commit: robot taskboard_environment, 23 links, 22 joints
Links:
- removed link ket41_link
- added link ket4_link, mass 0.01; collision mesh filename=package://project_description/meshes/taskboard_1/dae/KET4.d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; visual mesh filename=package://project_description/meshes/taskboard_1/dae/KET4.d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
Joints:
- joint bnc_male_joint: origin xyz=0.133 -0.214 0.011 rpy=3.14118 0 0 -> xyz=0.333 0.356 0.191 rpy=3.14118 0 0
- joint dsub_male_joint: origin xyz=0.166 -0.325 0.008 rpy=-1.571 0 0 -> xyz=0.366 0.245 0.188 rpy=-1.571 0 0
- joint gear_large_joint: origin xyz=0.078 -0.278 0.01 rpy=3.14118 0 -3.14118 -> xyz=0.278 0.292 0.19 rpy=3.14118 0 -3.14118
- joint gear_medium_joint: origin xyz=0.271 -0.314 0.01 rpy=3.14118 0 3.14118 -> xyz=0.471 0.256 0.19 rpy=3.14118 0 3.14118
- joint gear_small_joint: origin xyz=0.343 -0.259 0.01 rpy=-3.14118 0 -3.14118 -> xyz=0.543 0.311 0.19 rpy=-3.14118 0 -3.14118
- joint ket12_joint: origin xyz=0.059 -0.372 0.004 rpy=1.571 0 0 -> xyz=0.259 0.198 0.184 rpy=1.571 0 0
- joint ket16_joint: origin xyz=0.107 -0.171 0.025 rpy=0 0 0 -> xyz=0.307 0.399 0.205 rpy=0 0 0
- joint ket4_joint: child ket41_link -> ket4_link; origin xyz=0.347 -0.449 0.002 rpy=1.571 0 0 -> xyz=0.547 0.121 0.182 rpy=1.571 0 0
- joint ket8_joint: origin xyz=0.137 -0.413 0.004 rpy=0.000407 -1.57059 -0.000407 -> xyz=0.337 0.157 0.184 rpy=0.000407 -1.57059 -0.000407
- joint m12_nut_joint: origin xyz=0.341 -0.332 0.004 rpy=0 0 0 -> xyz=0.541 0.238 0.184 rpy=0 0 0
- joint m16_nut_joint: origin xyz=0.235 -0.432 0.012 rpy=-0.000407 1.57059 -0.000407 -> xyz=0.435 0.138 0.192 rpy=-0.000407 1.57059 -0.000407
- joint m4_nut_joint: origin xyz=0.052 -0.198 0.002 rpy=0 0 0 -> xyz=0.252 0.372 0.182 rpy=0 0 0
- joint m8_nut_joint: origin xyz=0.204 -0.251 0.003 rpy=0 0 0 -> xyz=0.404 0.319 0.183 rpy=0 0 0
- joint mcon_e10_sp_joint: origin xyz=0.30978 -0.17922 0.01978 rpy=0 0 0 -> xyz=0.50978 0.39078 0.19978 rpy=0 0 0
- joint rcog12_50_joint: origin xyz=0.194 -0.382 0.025 rpy=0 0 0 -> xyz=0.394 0.188 0.205 rpy=0 0 0
- joint rcog16_50_joint: origin xyz=0.276 -0.249 0.024 rpy=0 0 0 -> xyz=0.476 0.321 0.204 rpy=0 0 0
- joint rcog4_50_joint: origin xyz=0.196 -0.175 0.002 rpy=-0.01159 -1.57059 0.01159 -> xyz=0.396 0.395 0.182 rpy=-0.01159 -1.57059 0.01159
- joint rcog8_50_joint: origin xyz=0.065 -0.466 0.025 rpy=0 0 0 -> xyz=0.265 0.104 0.205 rpy=0 0 0
- joint rj45_male_joint: origin xyz=0.137 -0.479 0.00688 rpy=0 0 0 -> xyz=0.337 0.091 0.18688 rpy=0 0 0
- joint taskboard_joint: origin xyz=-0.2 -0.315 -0.0045 rpy=0 0 0 -> xyz=0.4 -0.25 0.1755 rpy=0 0 0
- joint tray_joint: origin xyz=0.2 -0.32 0 rpy=0 0 0 -> xyz=0.4 0.25 0.18 rpy=0 0 0
- joint usb_male_joint: origin xyz=0.294 -0.462 0.004 rpy=-1.571 0 -3.14118 -> xyz=0.494 0.108 0.184 rpy=-1.571 0 -3.141593

File: project_description/urdf/irb120_3_58/irb120_3_58_world.xacro (robot description, xacro)
@@ -1,11 +1,18 @@
 <?xml version="1.0"?>
 <robot xmlns:xacro="http://www.ros.org/wiki/xacro" name="irb120_assembly">
-  <!-- 1. Pure Robot + Gripper -->
-  <xacro:include filename="$(find project_description)/urdf/irb120_3_58/irb120_3_58_robot.urdf" />
-  <!-- 2. Root Frame -->
-  <joint name="world_to_robot" type="fixed">
-    <parent link="world" />
-    <child link="base_link" />
-    <origin xyz="0 0.32 0" rpy="0 0 0" />
-  </joint>
+<!-- Migrating to ABB1200 due to reach issue-->
+<!-- <xacro:include filename="$(find project_description)/urdf/irb120_3_58/irb120_3_58_robot.urdf" /> -->
+<xacro:include filename="$(find project_description)/urdf/irb1200_5_90/irb1200_5_90.urdf" />
+<link name="world"/>
+<joint name="world_to_robot" type="fixed">
+  <parent link="world" />
+  <child link="base_link" />
+  <origin xyz="0 0.32 0" rpy="0 0 0" />
+</joint>
+<link name="onrobot_2fg7_tcp" />
+<joint name="onrobot_2fg7_tcp_joint" type="fixed">
+  <parent link="gripper_base_link" />
+  <child link="onrobot_2fg7_tcp" />
+  <origin xyz="0 0 0.115" rpy="0 0 0" />
+</joint>
 </robot>
